Commit message: test

File: pr2_description/urdf/base_v0/base.transmission.xacro (robot description, xacro)
@@ -3,16 +3,26 @@
   <!--  Caster wheel transmission   -->
   <xacro:macro name="pr2_wheel_transmission_v0" params="suffix parent reflect">
-    <transmission type="pr2_mechanism_model/SimpleTransmission" name="${parent}_${suffix}_wheel_trans">
-      <actuator name="${parent}_${suffix}_wheel_motor" />
-      <joint name="${parent}_${suffix}_wheel_joint" />
-      <mechanicalReduction>${reflect * 624/35 * 80/18}</mechanicalReduction>
+    <transmission name="${parent}_${suffix}_wheel_trans">
+      <type>transmission_interface/SimpleTransmission</type>
+      <actuator name="${parent}_${suffix}_wheel_motor">
+        <mechanicalReduction>${reflect * 624/35 * 80/18}</mechanicalReduction>
+      </actuator>
+      <joint name="${parent}_${suffix}_wheel_joint">
+        <hardwareInterface>hardware_interface/VelocityJointInterface</hardwareInterface>
+        <hardwareInterface>hardware_interface/JointStateInterface</hardwareInterface>
+      </joint>
     </transmission>
   </xacro:macro>
   <!-- Hub transmission only -->
   <xacro:macro name="pr2_caster_transmission_v0" params="suffix">
-    <transmission type="pr2_mechanism_model/SimpleTransmission" name="${suffix}_rotation_trans">
-      <actuator name="${suffix}_rotation_motor" />
-      <joint name="${suffix}_rotation_joint" />
-      <mechanicalReduction>${-1 * 624/35 * 80/18}</mechanicalReduction>
+    <transmission name="${suffix}_rotation_trans">
+      <type>transmission_interface/SimpleTransmission</type>
+      <actuator name="${suffix}_rotation_motor">
+        <mechanicalReduction>${-1 * 624/35 * 80/18}</mechanicalReduction>
+      </actuator>
+      <joint name="${suffix}_rotation_joint">
+        <hardwareInterface>hardware_interface/VelocityJointInterface</hardwareInterface>
+        <hardwareInterface>hardware_interface/JointStateInterface</hardwareInterface>
+      </joint>
     </transmission>
   </xacro:macro>

File: pr2_description/urdf/forearm_v0/forearm.transmission.xacro (robot description, xacro)
@@ -3,9 +3,20 @@
   <xacro:macro name="pr2_forearm_transmission_v0" params="side">
     <!-- Wrist flex , Wrist roll -->
-    <transmission type="pr2_mechanism_model/WristTransmission" name="${side}_wrist_trans">
-      <rightActuator name="${side}_wrist_r_motor" mechanicalReduction="${624/35*54/16}"/>
-      <leftActuator name="${side}_wrist_l_motor"  mechanicalReduction="${624/35*54/16}"/>
-      <flexJoint name="${side}_wrist_flex_joint"  mechanicalReduction="-1.0" />
-      <rollJoint name="${side}_wrist_roll_joint"  mechanicalReduction="1.0" />
+    <transmission name="${side}_wrist_trans">
+      <type>transmission_interface/DifferentialTransmission</type>
+      <actuator name="${side}_wrist_r_motor">
+        <mechanicalReduction>${624/35*54/16}</mechanicalReduction>
+      </actuator>
+      <actuator name="${side}_wrist_l_motor">
+        <mechanicalReduction>${624/35*54/16}</mechanicalReduction>
+      </actuator>
+      <joint name="${side}_wrist_flex_joint">
+        <hardwareInterface>hardware_interface/PositionJointInterface</hardwareInterface>
+        <mechanicalReduction>-1.0</mechanicalReduction>
+      </joint>
+      <joint name="${side}_wrist_roll_joint">
+        <hardwareInterface>hardware_interface/PositionJointInterface</hardwareInterface>
+        <mechanicalReduction>1.0</mechanicalReduction>
+      </joint>
     </transmission>
   </xacro:macro>
